File: Schematics/MarsAquaAdapter/signalConditioner.sch (EAGLE design)
At the start: 19 parts, among them IC3 LMV358SOIC, Q2 MMBT4403

Commit message: Add pull down and update divider
Parts:
- added RC2VD1: 4.7k, SparkFun-Resistors:RESISTOR1206
- added RC2VU1: 330k, SparkFun-Resistors:RESISTOR1206
- RC2VD: value 18k -> 20k
Connections:
- new net N$2: RC2VD.1, RC2VD1.2
- net GND: now also RC2VD1.1, RC2VU1.1; no longer RC2VD.1
- net INPUT: now also RC2VU1.2
Changed lines of the file:
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@@
 <part name="U$1" library="SMD-RJ45" deviceset="MOLEX-RJ45-SMT" device=""/>
 <part name="J2" library="SparkFun-Connectors" deviceset="M04" device="LONGPADS"/>
-<part name="RC2VD" library="SparkFun-Resistors" deviceset="RESISTOR" device="1206" value="18k"/>
+<part name="RC2VD" library="SparkFun-Resistors" deviceset="RESISTOR" device="1206" value="20k"/>
 <part name="RC2VU" library="SparkFun-Resistors" deviceset="RESISTOR" device="1206" value="330k"/>
 <part name="R2" library="SparkFun-Resistors" deviceset="RESISTOR" device="1206" value="20k"/>
@@
 <part name="GND5" library="SparkFun-Aesthetics" deviceset="GND" device=""/>
 <part name="GND9" library="SparkFun-Aesthetics" deviceset="GND" device=""/>
+<part name="RC2VD1" library="SparkFun-Resistors" deviceset="RESISTOR" device="1206" value="4.7k"/>
+<part name="RC2VU1" library="SparkFun-Resistors" deviceset="RESISTOR" device="1206" value="330k"/>
+<part name="GND12" library="SparkFun-Aesthetics" deviceset="GND" device=""/>
 </parts>
 <sheets>
@@
 <instance part="C2" gate="G$1" x="63.5" y="20.32"/>
 <instance part="GND1" gate="1" x="111.76" y="71.12"/>
-<instance part="GND2" gate="1" x="106.68" y="20.32"/>
+<instance part="GND2" gate="1" x="106.68" y="7.62"/>
 <instance part="GND3" gate="1" x="63.5" y="15.24"/>
 <instance part="GND6" gate="1" x="76.2" y="12.7"/>
@@
 <instance part="GND5" gate="1" x="15.24" y="53.34"/>
 <instance part="GND9" gate="1" x="35.56" y="53.34"/>
+<instance part="RC2VD1" gate="G$1" x="106.68" y="17.78" rot="R90"/>
+<instance part="RC2VU1" gate="G$1" x="50.8" y="22.86" rot="R90"/>
+<instance part="GND12" gate="1" x="50.8" y="15.24"/>
 </instances>
 <busses>
@@
 </segment>
 <segment>
-<pinref part="RC2VD" gate="G$1" pin="1"/>
 <pinref part="GND2" gate="1" pin="GND"/>
+<wire x1="106.68" y1="10.16" x2="106.68" y2="12.7" width="0.1524" layer="91"/>
+<pinref part="RC2VD1" gate="G$1" pin="1"/>
 </segment>
 <segment>
@@
 <wire x1="15.24" y1="63.5" x2="35.56" y2="63.5" width="0.1524" layer="91"/>
 <wire x1="35.56" y1="63.5" x2="35.56" y2="55.88" width="0.1524" layer="91"/>
+</segment>
+<segment>
+<pinref part="RC2VU1" gate="G$1" pin="1"/>
+<pinref part="GND12" gate="1" pin="GND"/>
 </segment>
 </net>
@@
 <wire x1="45.72" y1="33.02" x2="45.72" y2="38.1" width="0.1524" layer="91"/>
 <wire x1="45.72" y1="43.18" x2="45.72" y2="38.1" width="0.1524" layer="91"/>
-</segment>
-</net>
+<pinref part="RC2VU1" gate="G$1" pin="2"/>
+<wire x1="50.8" y1="27.94" x2="50.8" y2="38.1" width="0.1524" layer="91"/>
+<junction x="50.8" y="38.1"/>
+</segment>
+</net>
+<net name="N$2" class="0">
+<segment>
+<pinref part="RC2VD" gate="G$1" pin="1"/>
+<pinref part="RC2VD1" gate="G$1" pin="2"/>
+</segment>
+</net>
