File: Schematics/PiBreakout328PBwithPH/breakoutWithPH.brd (EAGLE design)
At the start: 57.1 x 87.3 mm, 28 parts, among them J1 FEMALE 2x3, U1 PH_SMD, U2 ATMEGA328P_TQFP

Commit message: Temperature and PH firmware
Parts:
- added R5: 4.7k, SparkFun-Resistors:1206
- moved R4 2.93 mm to (12.7, 49.5)
Connections:
- net N$25: now also R5.2
- net N$26: now also R4.2
- net N$8: no longer R4.2
- net VDD: now also R5.1
Routing:
- net N$8: track 34.1 -> 14.9 mm
- net VDD: track 183.5 -> 185.5 mm
- net N$26: track 56.9 -> 58.1 mm
- net N$25: track 45.9 -> 46.8 mm
Changed lines of the file:
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@@
 <attribute name="VALUE" x="33.02" y="63.5" size="0.4064" layer="27" rot="R90"/>
 </element>
-<element name="R4" library="SparkFun-Resistors" package="1206" value="4.7k" x="15.494" y="50.419"/>
 <element name="J1" library="SparkFun-Connectors" package="2X3" value="FEMALE 2x3" x="38.1" y="76.2" rot="R90">
 <attribute name="PROD_ID" value="CONN-11566" x="38.1" y="76.2" size="1.778" layer="27" rot="R90" display="off"/>
@@
 <element name="C1" library="SparkFun-Capacitors" package="1206" value=".01uF" x="28.194" y="80.01" rot="R270"/>
 <element name="R3" library="SparkFun-Resistors" package="1206" value="10k" x="29.591" y="75.184" rot="R180"/>
+<element name="R4" library="SparkFun-Resistors" package="1206" value="4.7k" x="12.7" y="49.53"/>
+<element name="R5" library="SparkFun-Resistors" package="1206" value="4.7k" x="15.24" y="59.69"/>
 </elements>
 <signals>
@@
 <contactref element="U2" pad="4"/>
 <contactref element="U2" pad="18"/>
-<contactref element="R4" pad="1"/>
 <contactref element="C3" pad="2"/>
 <wire x1="5.08" y1="27.94" x2="7.62" y2="27.94" width="0.3048" layer="1"/>
@@
 <wire x1="26.27" y1="61.7474" x2="26.27" y2="65.64" width="0.3048" layer="1"/>
 <wire x1="7.62" y1="27.94" x2="8.89" y2="29.21" width="0.3048" layer="1"/>
-<wire x1="8.89" y1="29.21" x2="8.89" y2="50.8" width="0.3048" layer="1"/>
-<wire x1="8.89" y1="50.8" x2="8.89" y2="69.85" width="0.3048" layer="1"/>
+<wire x1="8.89" y1="29.21" x2="8.89" y2="49.53" width="0.3048" layer="1"/>
+<wire x1="8.89" y1="49.53" x2="8.89" y2="59.69" width="0.3048" layer="1"/>
+<wire x1="8.89" y1="59.69" x2="8.89" y2="69.85" width="0.3048" layer="1"/>
 <wire x1="21.59" y1="16.86" x2="21.59" y2="15.24" width="0.3048" layer="1"/>
 <wire x1="21.59" y1="15.24" x2="20.32" y2="13.97" width="0.3048" layer="1"/>
@@
 <wire x1="31.75" y1="71.12" x2="28.67" y2="68.04" width="0.3048" layer="1"/>
 <wire x1="28.67" y1="68.04" x2="26.27" y2="65.64" width="0.3048" layer="1"/>
-<wire x1="14.094" y1="50.419" x2="9.271" y2="50.419" width="0.3048" layer="1"/>
-<wire x1="9.271" y1="50.419" x2="8.89" y2="50.8" width="0.3048" layer="1"/>
 <wire x1="26.27" y1="65.64" x2="21.082" y2="60.452" width="0.3048" layer="1"/>
 <wire x1="21.082" y1="60.452" x2="21.082" y2="35.433" width="0.3048" layer="1"/>
@@
 <wire x1="30.991" y1="75.184" x2="30.991" y2="71.879" width="0.3048" layer="1"/>
 <wire x1="30.991" y1="71.879" x2="31.75" y2="71.12" width="0.3048" layer="1"/>
+<contactref element="R4" pad="1"/>
+<contactref element="R5" pad="1"/>
+<wire x1="11.3" y1="49.53" x2="8.89" y2="49.53" width="0.3048" layer="1"/>
+<wire x1="13.84" y1="59.69" x2="8.89" y2="59.69" width="0.3048" layer="1"/>
 </signal>
 <signal name="N$1">
@@
 <signal name="N$8">
 <contactref element="U2" pad="29"/>
-<contactref element="R4" pad="2"/>
-<wire x1="22.3774" y1="65.64" x2="19.92" y2="65.64" width="0.3048" layer="1"/>
-<wire x1="19.92" y1="65.64" x2="16.51" y2="62.23" width="0.3048" layer="1"/>
-<wire x1="16.51" y1="62.23" x2="16.51" y2="50.803" width="0.3048" layer="1"/>
-<wire x1="16.51" y1="50.803" x2="16.894" y2="50.419" width="0.3048" layer="1"/>
 <wire x1="24.13" y1="68.58" x2="24.13" y2="65.913" width="0.3048" layer="1"/>
 <wire x1="24.13" y1="65.913" x2="23.876" y2="65.659" width="0.3048" layer="1"/>
@@
 <wire x1="19.45" y1="66.44" x2="15.748" y2="62.738" width="0.3048" layer="1"/>
 <wire x1="15.748" y1="35.052" x2="17.78" y2="33.02" width="0.3048" layer="1"/>
-<wire x1="15.748" y1="35.052" x2="15.748" y2="62.738" width="0.3048" layer="1"/>
+<wire x1="15.748" y1="35.052" x2="15.748" y2="59.69" width="0.3048" layer="1"/>
+<wire x1="15.748" y1="59.69" x2="15.748" y2="62.738" width="0.3048" layer="1"/>
 <wire x1="17.78" y1="33.02" x2="20.32" y2="33.02" width="0.3048" layer="1"/>
 <wire x1="20.32" y1="33.02" x2="21.59" y2="31.75" width="0.3048" layer="1"/>
 <wire x1="21.59" y1="31.75" x2="21.59" y2="28.86" width="0.3048" layer="1"/>
+<contactref element="R5" pad="2"/>
+<wire x1="16.64" y1="59.69" x2="15.748" y2="59.69" width="0.3048" layer="1"/>
 </signal>
 <signal name="N$26">
@@
 <wire x1="22.3774" y1="67.24" x2="18.98" y2="67.24" width="0.3048" layer="1"/>
 <wire x1="18.98" y1="67.24" x2="15.24" y2="63.5" width="0.3048" layer="1"/>
-<wire x1="15.24" y1="63.5" x2="15.24" y2="17.78" width="0.3048" layer="1"/>
+<wire x1="15.24" y1="63.5" x2="15.24" y2="49.53" width="0.3048" layer="1"/>
+<wire x1="15.24" y1="49.53" x2="15.24" y2="17.78" width="0.3048" layer="1"/>
 <wire x1="15.24" y1="17.78" x2="16.51" y2="16.51" width="0.3048" layer="1"/>
 <wire x1="16.51" y1="16.51" x2="16.74" y2="16.51" width="0.3048" layer="1"/>
 <wire x1="16.74" y1="16.51" x2="17.09" y2="16.86" width="0.3048" layer="1"/>
+<contactref element="R4" pad="2"/>
+<wire x1="14.1" y1="49.53" x2="15.24" y2="49.53" width="0.3048" layer="1"/>
 </signal>
 <signal name="N$29">
